Commit message: Update inspire hand urdf, thumb moves, but still not fixed

File: src/inspire_hand_description/urdf/inspire_hand_right_parts.urdf (robot description, URDF)
Before this commit: robot inspire_hand_right, 10 links, 9 joints
Links:
- added link thumb_2_link, mass 0.01; collision mesh filename=package://inspire_hand_description/meshes/right/part_030.stl; visual mesh filename=package://inspire_hand_description/meshes/right/part_029.stl
- link base_link: geometry collision mesh filename=package://inspire_hand_description/meshes/right/part_032.stl; visual mesh filename=package://inspire_hand_description/meshes/right/part_000.stl
- link thumb_1_link: geometry collision mesh filename=package://inspire_hand_description/meshes/right/part_031.stl; visual mesh filename=package://inspire_hand_description/meshes/right/part_031.stl
Joints:
- added joint thumb_2_joint: type revolute, parent thumb_1_link, child thumb_2_link, origin xyz=-0.008 0.016 -0.044 rpy=0 0 0, axis 0 1 0, limit lower=0 upper=0.48 effort=50 velocity=1
- joint thumb_1_joint: axis -1 0 0 -> 0 0 -1; limit lower=0 upper=1.5 effort=50 velocity=1 -> lower=0 upper=1.246 effort=50 velocity=1; origin xyz=-0.0083 -0.0725 0.1118 rpy=0 0 0 -> xyz=-0.041 -0.02 0.09 rpy=0 0 0
