Commit message: inspire_hand_description: update hand model with new URDFs from Inspire support
- Update URDF files from DFTP source pack with integrated palm geometry
- Replace mesh files with new CAD exports (base_link now includes palm)
- Simplify RViz configs and fix fixed_frame to base_footprint
- Fix tactile_pointcloud_node.py to use DOF_RAW_CALIBRATION

The new model integrates palm geometry into base_link rather than
separate palm_1/palm_2 links, matching the DFTP force sensor design.

Signed-off-by: laurent-19 <laurentiu.popa@analog.com>

File: src/inspire_hand_description/urdf/rh56e2_left.urdf (robot description, URDF)
Before this commit: robot RH56E2_L_2025_9_10, 33 links, 32 joints
Links:
- removed link left_palm_1
- removed link left_palm_2
- link base_link: mass 0.090 -> 0.62266
- link left_index_1: mass 0.018690000000000002 -> 0.02841
- link left_index_2: mass 0.01102 -> 0.01218
- link left_index_force_sensor_1: mass 0.00020279 -> 0.001
- link left_index_force_sensor_2: mass 0.000255748193489171 -> 0.001
- link left_index_force_sensor_3: mass 6.79653902597574E-05 -> 0.001
- link left_little_1: mass 0.018690000000000002 -> 0.02841
- link left_little_2: mass 0.018690000000000002 -> 0.00957
- link left_little_force_sensor_1: mass 0.000202794502264302 -> 0.001
- link left_little_force_sensor_2: mass 0.00028024674848609 -> 0.001
- link left_little_force_sensor_3: mass 6.1053667014177E-05 -> 0.001
- link left_middle_1: mass 0.01866 -> 0.02841
- link left_middle_2: mass 0.01767 -> 0.01561
- link left_middle_force_sensor_1: mass 0.000202794522112893 -> 0.001
- link left_middle_force_sensor_2: mass 0.000262573593923136 -> 0.001
- link left_middle_force_sensor_3: mass 6.64914272946078E-05 -> 0.001
- link left_palm_force_sensor: mass 0.00240886556268154 -> 0.001
- link left_ring_1: mass 0.018690000000000002 -> 0.02841
- link left_ring_2: mass 0.01102 -> 0.01281
- link left_ring_force_sensor_1: mass 0.000202794434376476 -> 0.001
- link left_ring_force_sensor_2: mass 0.000255748190883527 -> 0.001
- link left_ring_force_sensor_3: mass 6.79657634628817E-05 -> 0.001
- link left_thumb_1: mass 0.01537 -> 0.00746
- link left_thumb_2: mass 0.11034000000000001 -> 0.04264
- link left_thumb_3: mass 0.01779 -> 0.01501
- link left_thumb_4: mass 0.00766 -> 0.00972
- link left_thumb_force_sensor_1: mass 0.000234351522411044 -> 0.001
- link left_thumb_force_sensor_2: mass 0.000119024235960817 -> 0.001
- link left_thumb_force_sensor_3: mass 0.000169894176021865 -> 0.001
- link left_thumb_force_sensor_4: mass 1.66991074236564E-05 -> 0.001
Joints:
- removed joint left_palm_1_joint
- removed joint left_palm_2_joint
- joint left_index_1_joint: axis 0 0 -1 -> 0 0 1; limit lower=0 upper=1.4381 effort=1 velocity=2 -> lower=0 upper=1.4381 effort=10 velocity=1; origin xyz=0.00056467 0.038679 -0.1564 rpy=-1.5359 0 0 -> xyz=0.038679 0.00056467 0.1564 rpy=1.5359 0 -1.5708
- joint left_index_2_joint: axis 0 0 -1 -> 0 0 1; limit lower=0 upper=1.476374 effort=1 velocity=2 -> lower=0 upper=3.14 effort=10 velocity=1; origin xyz=0.0034259 0.032596 -0.00055 rpy=0 0 0 -> xyz=-0.0034259 0.032596 0.00055 rpy=0 0 0
- joint left_index_force_sensor_1_joint: origin xyz=0.012046 0.019649 -0.006651 rpy=-1.5708 1.5351 -1.3587 -> xyz=-0.012046 0.019649 0.006651 rpy=1.5708 -1.5351 -1.7829
- joint left_index_force_sensor_2_joint: origin xyz=0.0081655 0.037446 -0.0060795 rpy=-0.037141 0 -0.34877 -> xyz=-0.0081655 0.037446 0.0060795 rpy=1.5708 -1.5337 -1.222
- joint left_index_force_sensor_3_joint: origin xyz=0.0086237 0.052572 -0.0060954 rpy=-1.5708 1.5252 -0.87237 -> xyz=-0.0086237 0.052572 0.0060954 rpy=1.5708 -1.5252 -2.2692
- joint left_little_1_joint: axis 0 0 -1 -> 0 0 1; limit lower=0 upper=1.4381 effort=1 velocity=2 -> lower=0 upper=1.4381 effort=10 velocity=1; origin xyz=0.00056467 -0.025916 -0.15365 rpy=-1.6755 0 0 -> xyz=-0.025916 0.00056467 0.15365 rpy=1.6755 0 -1.5708
- joint left_little_2_joint: axis 0 0 -1 -> 0 0 1; limit lower=0 upper=1.476374 effort=1 velocity=2 -> lower=0 upper=3.14 effort=10 velocity=1; origin xyz=0.0034259 0.032596 -0.00055 rpy=0 0 0 -> xyz=-0.0034259 0.032596 0.00055 rpy=0 0 0
- joint left_little_force_sensor_1_joint: origin xyz=0.012046 0.019649 -0.006651 rpy=1.5708 1.4637 1.7829 -> xyz=-0.012046 0.019649 0.006651 rpy=-1.5708 -1.4637 1.3587
- joint left_little_force_sensor_2_joint: origin xyz=0.0064514 0.027683 -0.0061172 rpy=1.5708 1.4597 1.2289 -> xyz=-0.0064514 0.027683 0.0061172 rpy=-1.5708 -1.4597 1.9127
- joint left_little_force_sensor_3_joint: origin xyz=0.0063973 0.042707 -0.0061154 rpy=1.5708 1.4336 2.2761 -> xyz=-0.0063973 0.042707 0.0061154 rpy=-1.5708 -1.4336 0.86551
- joint left_middle_1_joint: axis 0 0 -1 -> 0 0 1; limit lower=0 upper=1.4381 effort=1 velocity=2 -> lower=0 upper=1.4381 effort=10 velocity=1; origin xyz=0.00056467 0.0171 -0.157 rpy=-1.5708 0 0 -> xyz=0.0171 0.00056467 0.157 rpy=1.5708 0 -1.5708
- joint left_middle_2_joint: axis 0 0 -1 -> 0 0 1; limit lower=0 upper=1.476374 effort=1 velocity=2 -> lower=0 upper=3.14 effort=10 velocity=1; origin xyz=0.0034259 0.032596 -0.00055 rpy=0 0 0 -> xyz=-0.0034259 0.032596 0.00055 rpy=0 0 0
- joint left_middle_force_sensor_1_joint: origin xyz=0.012046 0.019649 -0.006651 rpy=-1.9353 1.5708 -1.7232 -> xyz=-0.012046 0.019649 0.006651 rpy=0.73473 -1.5708 -0.94682
- joint left_middle_force_sensor_2_joint: origin xyz=0.009086 0.040962 -0.0061003 rpy=-1.0917 1.5708 -1.4646 -> xyz=-0.009086 0.040962 0.0061003 rpy=1.8942 -1.5708 -1.5214
- joint left_middle_force_sensor_3_joint: origin xyz=0.0098294 0.056051 -0.0061006 rpy=-2.1401 1.5708 -1.4657 -> xyz=-0.0098294 0.056051 0.0061006 rpy=0.84662 -1.5708 -1.521
- joint left_palm_force_sensor_joint: origin xyz=0.012296 -0.00036819 0.088601 rpy=1.5708 0 1.5708 -> xyz=0.00036819 0.012296 0.1196 rpy=1.5708 0 3.1416; parent left_palm_1 -> base_link
- joint left_ring_1_joint: axis 0 0 -1 -> 0 0 1; limit lower=0 upper=1.4381 effort=1 velocity=2 -> lower=0 upper=1.4381 effort=10 velocity=1; origin xyz=0.00056467 -0.0045302 -0.15683 rpy=-1.6232 0 0 -> xyz=-0.0045302 0.00056467 0.15683 rpy=1.6232 0 -1.5708
- joint left_ring_2_joint: axis 0 0 -1 -> 0 0 1; limit lower=0 upper=1.476374 effort=1 velocity=2 -> lower=0 upper=3.14 effort=10 velocity=1; origin xyz=0.0034259 0.032596 -0.00055 rpy=0 0 0 -> xyz=-0.0034259 0.032596 0.00055 rpy=0 0 0
- joint left_ring_force_sensor_1_joint: origin xyz=0.012046 0.019649 -0.006651 rpy=1.5708 1.5172 1.7829 -> xyz=-0.012046 0.019649 0.006651 rpy=-1.5708 -1.5172 1.3587
- joint left_ring_force_sensor_2_joint: origin xyz=0.0081655 0.037446 -0.0060795 rpy=1.5708 1.5151 1.222 -> xyz=-0.0081655 0.037446 0.0060795 rpy=-1.5708 -1.5151 1.9196
- joint left_ring_force_sensor_3_joint: origin xyz=0.0086237 0.052572 -0.0060954 rpy=1.5708 1.5025 2.2692 -> xyz=-0.0086237 0.052572 0.0060954 rpy=-1.5708 -1.5025 0.87237
- joint left_thumb_1_joint: limit lower=0 upper=1.658 effort=1 velocity=2 -> lower=0 upper=1.1641 effort=10 velocity=1; origin xyz=0.02101 0.0269 -0.0826 rpy=3.1416 0 0 -> xyz=0.0269 0.02101 0.0689 rpy=0 0 0
- joint left_thumb_2_joint: axis 0.17365 0 0.98481 -> 0 0 -1; limit lower=0 upper=0.62 effort=1 velocity=2 -> lower=0 upper=0.5864 effort=10 velocity=1; origin xyz=0.013438 -0.012862 -0.0076 rpy=1.5708 0 -1.5708 -> xyz=0.0073431 0.011232 0.0052 rpy=1.5708 0 -2.8798
- joint left_thumb_3_joint: axis 0.17365 0 0.98481 -> 0 0 -1; limit lower=0 upper=0.5410520681182421 effort=1 velocity=2 -> lower=0 upper=0.5 effort=10 velocity=1; mimic joint=left_thumb_2_joint multiplier=0.8392 offset=0 -> joint=left_thumb_2_joint multiplier=0.8024 offset=0; origin xyz=0.052954 0.032799 -0.0093372 rpy=0 0 0 -> xyz=-0.031403 0.021069 -0.001299 rpy=0 0 0
- joint left_thumb_4_joint: axis 0.17365 0 0.98481 -> 0 0 -1; limit lower=0 upper=0.45553093477052004 effort=1 velocity=2 -> lower=0 upper=3.14 effort=10 velocity=1; mimic joint=left_thumb_3_joint multiplier=0.891 offset=0 -> joint=left_thumb_3_joint multiplier=0.9487 offset=0; origin xyz=0.01865 0.013373 -0.0022731 rpy=0 0 0 -> xyz=-0.021903 0.012816 -0.0003 rpy=0 0 0
- joint left_thumb_force_sensor_1_joint: origin xyz=0.023412 0.033251 0.0070079 rpy=1.1285 1.3976 3.1383 -> xyz=-0.0087121 0.026305 -0.0089605 rpy=1.2213 -1.5708 -3.14
- joint left_thumb_force_sensor_2_joint: origin xyz=0.0080283 0.016443 0.00982 rpy=0.96258 1.4071 3.0993 -> xyz=-0.011771 0.01699 -0.0077514 rpy=-1.8405 -1.5705 0
- joint left_thumb_force_sensor_3_joint: origin xyz=0.0076349 0.020486 0.0088094 rpy=0.64092 1.3963 -3.1415 -> xyz=-0.014598 0.014721 -0.0073103 rpy=0.18602 -1.5708 -2.2971
- joint left_thumb_force_sensor_4_joint: origin xyz=0.018831 0.027914 0.0068352 rpy=1.7521 1.3962 -3.1401 -> xyz=-0.028987 0.017301 -0.0073513 rpy=2.0775 1.5708 -2.12

File: src/inspire_hand_description/urdf/rh56e2_right.urdf (robot description, URDF)
Before this commit: robot RH56E2_R_2025_9_11, 33 links, 32 joints
Links:
- removed link right_palm_1
- removed link right_palm_2
- link base_link: mass 0.090 -> 0.62266
- link right_index_1: mass 0.018690000000000002 -> 0.02841
- link right_index_2: mass 0.01102 -> 0.01218
- link right_index_force_sensor_1: mass 0.00020277926206694 -> 0.001
- link right_index_force_sensor_2: mass 0.000255748458180208 -> 0.001
- link right_index_force_sensor_3: mass 6.79646984897729E-05 -> 0.001
- link right_little_1: mass 0.018690000000000002 -> 0.02841
- link right_little_2: mass 0.01166 -> 0.00957
- link right_little_force_sensor_1: mass 0.000202779290224811 -> 0.001
- link right_little_force_sensor_2: mass 0.000280265363825451 -> 0.001
- link right_little_force_sensor_3: mass 6.10539921684107E-05 -> 0.001
- link right_middle_1: mass 0.01866 -> 0.02841
- link right_middle_2: mass 0.01767 -> 0.01561
- link right_middle_force_sensor_1: mass 0.000202779388301744 -> 0.001
- link right_middle_force_sensor_2: mass 0.00026259331441686 -> 0.001
- link right_middle_force_sensor_3: mass 6.64914575467581E-05 -> 0.001
- link right_palm_force_sensor: mass 0.00240887838334331 -> 0.001
- link right_ring_1: mass 0.018690000000000002 -> 0.02841
- link right_ring_2: mass 0.01102 -> 0.01281
- link right_ring_force_sensor_1: mass 0.00020277922338036 -> 0.001
- link right_ring_force_sensor_2: mass 0.00025574845564278 -> 0.001
- link right_ring_force_sensor_3: mass 6.79650392240318E-05 -> 0.001
- link right_thumb_1: mass 0.01537 -> 0.00746
- link right_thumb_2: mass 0.11034000000000001 -> 0.04264
- link right_thumb_3: mass 0.01779 -> 0.01501
- link right_thumb_4: mass 0.00766 -> 0.00972
- link right_thumb_force_sensor_1: mass 0.000234345870584151 -> 0.001
- link right_thumb_force_sensor_2: mass 0.000119024197892742 -> 0.001
- link right_thumb_force_sensor_3: mass 0.000169893832350009 -> 0.001
- link right_thumb_force_sensor_4: mass 1.66991205082657E-05 -> 0.001
Joints:
- removed joint right_palm_1_joint
- removed joint right_palm_2_joint
- joint right_index_1_joint: axis 0 0 -1 -> 0 0 1; limit lower=0 upper=1.4381 effort=1 velocity=1 -> lower=0 upper=1.4381 effort=10 velocity=1; origin xyz=0.00056467 -0.038679 -0.1564 rpy=-1.6057 0 0 -> xyz=-0.038679 0.00056467 0.1564 rpy=1.6057 0 -1.5708
- joint right_index_2_joint: axis 0 0 -1 -> 0 0 1; limit lower=0 upper=1.476374 effort=1 velocity=1 -> lower=0 upper=3.14 effort=10 velocity=1; origin xyz=0.0034259 0.032596 0.00055 rpy=0 0 0 -> xyz=-0.0034259 0.032596 -0.00055 rpy=0 0 0
- joint right_index_force_sensor_1_joint: origin xyz=0.012046 0.019649 0.006651 rpy=1.5708 1.5351 1.7829 -> xyz=-0.012046 0.019649 -0.006651 rpy=-1.5708 -1.5351 1.3587
- joint right_index_force_sensor_2_joint: origin xyz=0.0081655 0.037446 0.0060795 rpy=1.5708 1.5337 1.222 -> xyz=-0.0081655 0.037446 -0.0060795 rpy=-1.5708 -1.5337 1.9196
- joint right_index_force_sensor_3_joint: origin xyz=0.0086237 0.052572 0.0060954 rpy=1.5708 1.5252 2.2692 -> xyz=-0.0086237 0.052572 -0.0060954 rpy=-1.5708 -1.5252 0.87237
- joint right_little_1_joint: axis 0 0 -1 -> 0 0 1; limit lower=0 upper=1.4381 effort=1 velocity=1 -> lower=0 upper=1.4381 effort=10 velocity=1; origin xyz=0.00056467 0.025916 -0.15365 rpy=-1.4661 0 0 -> xyz=0.025916 0.00056467 0.15365 rpy=1.4661 0 -1.5708
- joint right_little_2_joint: axis 0 0 -1 -> 0 0 1; limit lower=0 upper=1.476374 effort=1 velocity=1 -> lower=0 upper=3.14 effort=10 velocity=1; origin xyz=0.0034259 0.032596 0.00055 rpy=0 0 0 -> xyz=-0.0034259 0.032596 -0.00055 rpy=0 0 0
- joint right_little_force_sensor_1_joint: origin xyz=0.012046 0.019649 0.006651 rpy=-1.5708 1.4637 -1.3587 -> xyz=-0.0120461582060113 0.0196485471789908 -0.00665098451502223 rpy=1.5707963267949 -1.4636944932668 -1.78288465285966
- joint right_little_force_sensor_2_joint: origin xyz=0.0064512 0.027683 0.0061172 rpy=-1.5708 1.4597 -1.9127 -> xyz=-0.00645123763174135 0.0276833479200767 -0.00611719352979621 rpy=1.57079632679488 -1.45969392221055 -1.22888814145719
- joint right_little_force_sensor_3_joint: origin xyz=0.0063972 0.042707 0.0061154 rpy=-1.5708 1.4336 -0.86551 -> xyz=-0.00639723214432697 0.042706921918282 -0.00611537168168175 rpy=1.5707963267949 -1.43362674619531 -2.2760856926538
- joint right_middle_1_joint: axis 0 0 -1 -> 0 0 1; limit lower=0 upper=1.4381 effort=1 velocity=1 -> lower=0 upper=1.4381 effort=10 velocity=1; origin xyz=0.00056467 -0.0171 -0.157 rpy=-1.5708 0 0 -> xyz=-0.0171 0.00056467 0.157 rpy=1.5708 0 -1.5708
- joint right_middle_2_joint: axis 0 0 -1 -> 0 0 1; limit lower=0 upper=1.476374 effort=1 velocity=1 -> lower=0 upper=3.14 effort=10 velocity=1; origin xyz=0.0034259 0.032596 0.00055 rpy=0 0 0 -> xyz=-0.0034259 0.032596 -0.00055 rpy=0 0 0
- joint right_middle_force_sensor_1_joint: origin xyz=0.012046 0.019649 0.006651 rpy=-0.21209 1.5708 0 -> xyz=-0.012046 0.019649 -0.006651 rpy=2.9295 -1.5708 3.14
- joint right_middle_force_sensor_2_joint: origin xyz=0.0090859 0.040963 0.0061003 rpy=0.37285 1.5708 0 -> xyz=-0.0090859 0.040963 -0.0061003 rpy=2.7687 -1.5708 3.885
- joint right_middle_force_sensor_3_joint: origin xyz=0.0098294 0.056051 0.0061006 rpy=-0.67435 1.5708 0 -> xyz=-0.0098294 0.056051 -0.0061006 rpy=2.4672 -1.5708 3.14
- joint right_palm_force_sensor_joint: origin xyz=0.012296 0.00036819 0.089101 rpy=1.5708 0 1.5708 -> xyz=-0.00036819 0.012296 0.1196 rpy=1.5708 0 -3.1416; parent right_palm_1 -> base_link
- joint right_ring_1_joint: axis 0 0 -1 -> 0 0 1; limit lower=0 upper=1.4381 effort=1 velocity=1 -> lower=0 upper=1.4381 effort=10 velocity=1; origin xyz=0.00056467 0.0045302 -0.15683 rpy=-1.5184 0 0 -> xyz=0.0045302 0.00056467 0.15683 rpy=1.5184 0 -1.5708
- joint right_ring_2_joint: axis 0 0 -1 -> 0 0 1; limit lower=0 upper=1.476374 effort=1 velocity=1 -> lower=0 upper=3.14 effort=10 velocity=1; origin xyz=0.0034259 0.032596 0.00055 rpy=0 0 0 -> xyz=-0.0034259 0.032596 -0.00055 rpy=0 0 0
- joint right_ring_force_sensor_1_joint: origin xyz=0.012046 0.019649 0.006651 rpy=-1.5708 1.5172 -1.3587 -> xyz=-0.0120461582060112 0.019648547178991 -0.00665098451502209 rpy=1.57079632679491 -1.51723862304532 -1.78288465285967
- joint right_ring_force_sensor_2_joint: origin xyz=0.0081655 0.037446 0.0060795 rpy=-1.5708 1.5151 -1.9196 -> xyz=-0.00816549212353353 0.0374457610846523 -0.00607949056508933 rpy=1.57079632679487 -1.51508890383765 -1.22202982373572
- joint right_ring_force_sensor_3_joint: origin xyz=0.0086237 0.052572 0.0060954 rpy=-1.5708 1.5025 -0.87237 -> xyz=-0.00862372785817732 0.0525719273258207 -0.00609538761271226 rpy=1.57079632679487 -1.50247215376038 -2.26922737493233
- joint right_thumb_1_joint: limit lower=0 upper=1.658 effort=1 velocity=2 -> lower=0 upper=1.1641 effort=10 velocity=1; origin xyz=0.02101 -0.0269 -0.0826 rpy=-3.1416 0 0 -> xyz=-0.0269 0.02101 0.0689 rpy=0 0 0
- joint right_thumb_2_joint: axis 0.17365 0 -0.98481 -> 0 0 1; limit lower=0 upper=0.62 effort=1 velocity=2 -> lower=0 upper=0.5864 effort=10 velocity=1; origin xyz=0.013438 0.012862 -0.0076 rpy=1.5708 0 -1.5708 -> xyz=-0.0079252 0.0090599 0.0052 rpy=1.5708 0 2.8798
- joint right_thumb_3_joint: axis 0.17365 0 -0.98481 -> 0 0 1; limit lower=0 upper=0.5410520681182421 effort=1 velocity=2 -> lower=0 upper=0.5 effort=10 velocity=1; mimic joint=right_thumb_2_joint multiplier=0.8392 offset=0 -> joint=right_thumb_2_joint multiplier=0.8024 offset=0; origin xyz=-0.052954 0.032799 -0.0093372 rpy=0 0 0 -> xyz=0.031403 0.021069 0.00095 rpy=0 0 0
- joint right_thumb_4_joint: axis 0.17365 0 -0.98481 -> 0 0 1; limit lower=0 upper=0.45553093477052004 effort=1 velocity=2 -> lower=0 upper=3.14 effort=10 velocity=1; mimic joint=right_thumb_3_joint multiplier=0.891 offset=0 -> joint=right_thumb_3_joint multiplier=0.9487 offset=0; origin xyz=-0.01865 0.013373 -0.0022731 rpy=0 0 0 -> xyz=0.021903 0.012816 -0.0003 rpy=0 0 0
- joint right_thumb_force_sensor_1_joint: origin xyz=-0.023424 0.033251 0.007073 rpy=-0.99905 1.4338 0.13409 -> xyz=0.0087121 0.026305 -0.0067115 rpy=-1.5728 -1.5708 0.35156
- joint right_thumb_force_sensor_2_joint: origin xyz=-0.0080057 0.016443 0.0096921 rpy=-1.041 1.3851 -0.037357 -> xyz=0.011771 0.01699 -0.0077514 rpy=1.8405 -1.5705 3.1416
- joint right_thumb_force_sensor_3_joint: origin xyz=-0.0076345 0.020486 0.0088067 rpy=-0.64083 1.3963 4.2914E-05 -> xyz=0.014598 0.01472 -0.0073103 rpy=-0.20892 -1.5708 -0.81953
- joint right_thumb_force_sensor_4_joint: origin xyz=-0.01883 0.027914 0.0068326 rpy=-1.7492 1.3963 0.0014317 -> xyz=0.028987 0.017301 -0.0073512 rpy=1.6795 1.5708 2.7448
